File: KiCad/RubberBandGun.sch (KiCad schematic (older format))
At the start: 15 parts

Commit message: updates to schematic, remove some GradCap stuff
Connections:
- wire segments 80 -> 68
Changed lines of the file:
@@
 LIBS:mdoLibrary
 LIBS:Arduino_Nano-cache
+LIBS:RubberBandGun-cache
 EELAYER 25 0
 EELAYER END
@@
 L R R?
 U 1 1 5A767559
-P 7100 1250
-F 0 "R?" V 7180 1250 50  0000 C CNN
-F 1 "10K" V 7100 1250 50  0000 C CNN
-F 2 "" V 7030 1250 30  0000 C CNN
-F 3 "" H 7100 1250 30  0000 C CNN
-	1    7100 1250
-	1    0    0    -1
-$EndComp
-$Comp
-L ARD_of_4 A?
-U 1 1 5A7681AD
-P 7800 3850
-F 0 "A?" H 7800 3850 60  0000 C CNN
-F 1 "ARD_of_2" H 7800 3950 60  0000 C CNN
-F 2 "" H 7800 3850 60  0001 C CNN
-F 3 "" H 7800 3850 60  0001 C CNN
-	1    7800 3850
+P 4200 1250
+F 0 "R?" V 4280 1250 50  0000 C CNN
+F 1 "10K" V 4200 1250 50  0000 C CNN
+F 2 "" V 4130 1250 30  0000 C CNN
+F 3 "" H 4200 1250 30  0000 C CNN
+	1    4200 1250
 	1    0    0    -1
 $EndComp
@@
 Wire Wire Line
 	4900 700  9300 700
-Wire Wire Line
-	3200 950  7100 950
-Wire Wire Line
-	6800 950  6800 4350
-Wire Wire Line
-	6800 2000 6550 2000
 Wire Wire Line
 	5350 2300 3600 2300
@@
 	9750 1850 9850 1850
 Connection ~ 9850 1850
-Wire Wire Line
-	7100 950  7100 1100
-Connection ~ 6800 950
-Wire Wire Line
-	3600 3650 7350 3650
-Connection ~ 4000 3650
-Connection ~ 3800 3650
-Connection ~ 3600 3650
-Wire Wire Line
-	7100 1400 7100 3650
-Connection ~ 7100 3650
-Wire Wire Line
-	5350 3100 5250 3100
-Wire Wire Line
-	5250 3100 5250 3300
-Wire Wire Line
-	5250 3300 8250 3300
-Connection ~ 7100 3300
-Wire Wire Line
-	7350 4050 7250 4050
-Wire Wire Line
-	5350 3000 5150 3000
-Wire Wire Line
-	5150 3000 5150 3450
-Wire Wire Line
-	5150 3450 7100 3450
-Connection ~ 7100 3450
 $Sheet
 S 2150 7250 500  150
@@
 Connection ~ 5600 6400
 Wire Wire Line
-	6550 3000 6950 3000
-Wire Wire Line
-	6950 3000 6950 4550
-Wire Wire Line
-	6950 4550 6800 4550
-Wire Wire Line
 	5350 2700 4450 2700
 Wire Wire Line
@@
 Wire Wire Line
 	7100 4950 6800 4950
-Connection ~ 6800 2000
-Wire Wire Line
-	7250 4050 7250 4300
-Wire Wire Line
-	7250 4300 8250 4300
-Wire Wire Line
-	8250 4300 8250 3300
 Wire Wire Line
 	6800 4450 7700 4450
@@
 Wire Wire Line
 	4300 2600 5350 2600
+$Comp
+L ARD_of_4 A?
+U 1 1 5A7681AD
+P 7850 3600
+F 0 "A?" H 7850 3600 60  0000 C CNN
+F 1 "ARD_of_2" H 7850 3700 60  0000 C CNN
+F 2 "" H 7850 3600 60  0001 C CNN
+F 3 "" H 7850 3600 60  0001 C CNN
+	1    7850 3600
+	1    0    0    -1
+$EndComp
+Wire Wire Line
+	6550 3000 7000 3000
+Wire Wire Line
+	7000 3000 7000 4550
+Wire Wire Line
+	7000 4550 6800 4550
+Wire Wire Line
+	7400 3800 3600 3800
+Connection ~ 3600 3800
+Wire Wire Line
+	6550 2000 7400 2000
+Wire Wire Line
+	7400 950  7400 3400
+Wire Wire Line
+	3200 950  7400 950
+Connection ~ 7400 2000
+Connection ~ 3800 3800
+Connection ~ 4000 3800
 $EndSCHEMATC

Commit message: first cut wiring diagram
Parts:
- added L?: L, symbol L
- added R?: 10K, symbol R
- added SW? (x2): SW_PUSH, symbol SW_Push
Connections:
- wire segments 68 -> 84
Other:
- note added: "7.4 Volts"
- note added: "solenoid\ndriver"
Changed lines of the file:
@@
 	1    0    0    -1
 $EndComp
-Connection ~ 3050 6400
-Wire Wire Line
-	1250 6000 1250 5550
-Wire Wire Line
-	1550 6000 1250 6000
-Wire Wire Line
-	1250 6400 1250 6950
-Wire Wire Line
-	1550 6400 1250 6400
-Wire Wire Line
-	9850 6400 2750 6400
-Wire Wire Line
-	9850 1800 9850 6400
-Wire Wire Line
-	3050 4600 3050 6400
-Wire Wire Line
-	2750 4600 3050 4600
-Wire Wire Line
-	1250 4200 1550 4200
-Wire Wire Line
-	1250 3850 1250 4200
-Wire Wire Line
-	1250 4600 1550 4600
-Wire Wire Line
-	1250 4950 1250 4600
-Wire Wire Line
-	3200 4200 2750 4200
-Wire Wire Line
-	3200 950  3200 4200
-Connection ~ 3400 6400
-Wire Wire Line
-	3400 6400 3400 2000
-Wire Wire Line
-	3400 2000 5350 2000
-Wire Wire Line
-	5050 2200 4900 2200
-Wire Wire Line
-	4900 2200 4900 700
-Wire Wire Line
-	4900 700  9300 700
-Wire Wire Line
-	5350 2300 3600 2300
-Wire Wire Line
-	3600 1400 3600 4000
-Wire Wire Line
-	5350 2400 3800 2400
-Wire Wire Line
-	3800 1400 3800 4700
-Wire Wire Line
-	5350 2500 4000 2500
-Wire Wire Line
-	4000 1400 4000 4000
-Wire Wire Line
-	3600 4600 3600 6400
-Connection ~ 3600 6400
-Wire Wire Line
-	3800 5300 3800 6400
-Connection ~ 3800 6400
-Wire Wire Line
-	4000 4600 4000 6400
-Connection ~ 4000 6400
-Wire Wire Line
-	3600 1100 3600 950
-Connection ~ 3600 950
-Wire Wire Line
-	3800 1100 3800 950
-Connection ~ 3800 950
-Wire Wire Line
-	4000 1100 4000 950
-Connection ~ 4000 950
-Connection ~ 3600 2300
-Connection ~ 3800 2400
-Connection ~ 4000 2500
-Wire Wire Line
-	2750 6000 9950 6000
-Wire Wire Line
-	9950 6000 9950 1800
-Wire Wire Line
-	9300 700  9300 1950
-Wire Wire Line
-	9300 1950 10050 1950
-Wire Wire Line
-	10050 1950 10050 1800
-Wire Wire Line
-	9750 1800 9750 1850
-Wire Wire Line
-	9750 1850 9850 1850
-Connection ~ 9850 1850
 $Sheet
 S 2150 7250 500  150
@@
 	-1   0    0    -1
 $EndComp
-Wire Wire Line
-	5500 4550 5600 4550
-Wire Wire Line
-	5500 4650 5600 4650
-Wire Wire Line
-	5600 5050 5600 6400
-Connection ~ 5600 6400
-Wire Wire Line
-	5350 2700 4450 2700
-Wire Wire Line
-	4450 2700 4450 5700
-Wire Wire Line
-	4450 5700 7500 5700
-Wire Wire Line
-	7500 5700 7500 4750
-Wire Wire Line
-	7500 4750 6800 4750
-Wire Wire Line
-	5350 2800 4600 2800
-Wire Wire Line
-	4600 2800 4600 5550
-Wire Wire Line
-	4600 5550 7300 5550
-Wire Wire Line
-	7300 5550 7300 4850
-Wire Wire Line
-	7300 4850 6800 4850
-Wire Wire Line
-	5350 2900 4750 2900
-Wire Wire Line
-	4750 2900 4750 5400
-Wire Wire Line
-	4750 5400 7100 5400
-Wire Wire Line
-	7100 5400 7100 4950
-Wire Wire Line
-	7100 4950 6800 4950
-Wire Wire Line
-	6800 4450 7700 4450
-Wire Wire Line
-	7700 4450 7700 5850
-Wire Wire Line
-	7700 5850 4300 5850
-Wire Wire Line
-	4300 5850 4300 2600
-Wire Wire Line
-	4300 2600 5350 2600
 $Comp
 L ARD_of_4 A?
@@
 	1    0    0    -1
 $EndComp
+$Comp
+L SW_Push SW?
+U 1 1 5D7D1785
+P 4200 5050
+F 0 "SW?" H 4350 5160 50  0000 C CNN
+F 1 "SW_PUSH" H 4200 4970 50  0000 C CNN
+F 2 "" H 4200 5050 60  0000 C CNN
+F 3 "" H 4200 5050 60  0000 C CNN
+	1    4200 5050
+	0    -1   -1   0
+$EndComp
+$Comp
+L R R?
+U 1 1 5D7D3856
+P 4400 1250
+F 0 "R?" V 4480 1250 50  0000 C CNN
+F 1 "10K" V 4400 1250 50  0000 C CNN
+F 2 "" V 4330 1250 30  0000 C CNN
+F 3 "" H 4400 1250 30  0000 C CNN
+	1    4400 1250
+	1    0    0    -1
+$EndComp
+$Comp
+L SW_Push SW?
+U 1 1 5D7D389D
+P 4400 4300
+F 0 "SW?" H 4550 4410 50  0000 C CNN
+F 1 "SW_PUSH" H 4400 4220 50  0000 C CNN
+F 2 "" H 4400 4300 60  0000 C CNN
+F 3 "" H 4400 4300 60  0000 C CNN
+	1    4400 4300
+	0    -1   -1   0
+$EndComp
+$Comp
+L L L?
+U 1 1 5D7D3BAD
+P 8900 2950
+F 0 "L?" V 8850 2950 50  0000 C CNN
+F 1 "L" V 8975 2950 50  0000 C CNN
+F 2 "" H 8900 2950 50  0001 C CNN
+F 3 "" H 8900 2950 50  0001 C CNN
+	1    8900 2950
+	1    0    0    -1
+$EndComp
+Text Notes 8650 2400 1    118  ~ 0
+solenoid\ndriver
+Connection ~ 3050 6400
+Wire Wire Line
+	1250 6000 1250 5550
+Wire Wire Line
+	1550 6000 1250 6000
+Wire Wire Line
+	1250 6400 1250 6950
+Wire Wire Line
+	1550 6400 1250 6400
+Wire Wire Line
+	9850 6400 2750 6400
+Wire Wire Line
+	9850 1800 9850 6400
+Wire Wire Line
+	3050 4600 3050 6400
+Wire Wire Line
+	2750 4600 3050 4600
+Wire Wire Line
+	1250 4200 1550 4200
+Wire Wire Line
+	1250 3850 1250 4200
+Wire Wire Line
+	1250 4600 1550 4600
+Wire Wire Line
+	1250 4950 1250 4600
+Wire Wire Line
+	3200 4200 2750 4200
+Wire Wire Line
+	3200 950  3200 4200
+Connection ~ 3400 6400
+Wire Wire Line
+	3400 6400 3400 2000
+Wire Wire Line
+	3400 2000 5350 2000
+Wire Wire Line
+	5050 2200 4900 2200
+Wire Wire Line
+	4900 2200 4900 700
+Wire Wire Line
+	4900 700  9300 700
+Wire Wire Line
+	5350 2300 3600 2300
+Wire Wire Line
+	3600 1400 3600 4000
+Wire Wire Line
+	5350 2400 3800 2400
+Wire Wire Line
+	3800 1400 3800 4700
+Wire Wire Line
+	5350 2500 4000 2500
+Wire Wire Line
+	4000 1400 4000 4000
+Wire Wire Line
+	3600 4600 3600 6400
+Connection ~ 3600 6400
+Wire Wire Line
+	3800 5300 3800 6400
+Connection ~ 3800 6400
+Wire Wire Line
+	4000 4600 4000 6400
+Connection ~ 4000 6400
+Wire Wire Line
+	3600 1100 3600 950
+Connection ~ 3600 950
+Wire Wire Line
+	3800 1100 3800 950
+Connection ~ 3800 950
+Wire Wire Line
+	4000 1100 4000 950
+Connection ~ 4000 950
+Connection ~ 3600 2300
+Connection ~ 3800 2400
+Connection ~ 4000 2500
+Wire Wire Line
+	2750 6000 9950 6000
+Wire Wire Line
+	9950 6000 9950 1800
+Wire Wire Line
+	9300 700  9300 1950
+Wire Wire Line
+	9300 1950 10050 1950
+Wire Wire Line
+	10050 1950 10050 1800
+Wire Wire Line
+	9750 1800 9750 1850
+Wire Wire Line
+	9750 1850 9850 1850
+Connection ~ 9850 1850
+Wire Wire Line
+	5500 4550 5600 4550
+Wire Wire Line
+	5500 4650 5600 4650
+Wire Wire Line
+	5600 5050 5600 6400
+Connection ~ 5600 6400
+Wire Wire Line
+	7500 5700 7500 4750
+Wire Wire Line
+	7500 4750 6800 4750
+Wire Wire Line
+	7300 5550 7300 4850
+Wire Wire Line
+	7300 4850 6800 4850
+Wire Wire Line
+	7100 5400 7100 4950
+Wire Wire Line
+	7100 4950 6800 4950
+Wire Wire Line
+	6800 4450 7700 4450
+Wire Wire Line
+	7700 4450 7700 5850
 Wire Wire Line
 	6550 3000 7000 3000
@@
 Connection ~ 3800 3800
 Connection ~ 4000 3800
+Wire Wire Line
+	7300 4450 7300 3800
+Connection ~ 7300 3800
+Connection ~ 7300 4450
+Wire Wire Line
+	4950 5400 4950 3100
+Wire Wire Line
+	7100 5400 4950 5400
+Wire Wire Line
+	4950 3100 5350 3100
+Wire Wire Line
+	4850 5550 4850 3000
+Wire Wire Line
+	7300 5550 4850 5550
+Wire Wire Line
+	4850 3000 5350 3000
+Wire Wire Line
+	4750 5700 4750 2900
+Wire Wire Line
+	4750 5700 7500 5700
+Wire Wire Line
+	4750 2900 5350 2900
+Wire Wire Line
+	4650 5850 4650 2800
+Wire Wire Line
+	4650 2800 5350 2800
+Wire Wire Line
+	7700 5850 4650 5850
+Wire Wire Line
+	4200 1100 4200 950
+Connection ~ 4200 950
+Wire Wire Line
+	4200 1400 4200 4850
+Wire Wire Line
+	4200 5250 4200 6400
+Connection ~ 4200 6400
+Wire Wire Line
+	5350 2600 4200 2600
+Connection ~ 4200 2600
+Wire Wire Line
+	4400 1100 4400 950
+Connection ~ 4400 950
+Wire Wire Line
+	4400 1400 4400 4100
+Wire Wire Line
+	4400 4500 4400 6400
+Connection ~ 4400 6400
+Wire Wire Line
+	5350 2700 4400 2700
+Connection ~ 4400 2700
+Wire Notes Line
+	8350 2550 8350 2850
+Wire Notes Line
+	8350 2850 8650 2850
+Wire Notes Line
+	8650 2850 8650 2550
+Wire Notes Line
+	8650 2550 8350 2550
+Wire Wire Line
+	7400 2600 8350 2600
+Connection ~ 7400 2600
+Wire Wire Line
+	6550 3100 7500 3100
+Wire Wire Line
+	7500 3100 7500 2800
+Wire Wire Line
+	7500 2800 8350 2800
+Wire Wire Line
+	8900 2800 8900 2700
+Wire Wire Line
+	8900 2700 8650 2700
+Wire Wire Line
+	8900 3100 8900 6400
+Connection ~ 8900 6400
+Text Notes 900  3500 0    118  ~ 0
+7.4 Volts
 $EndSCHEMATC

Commit message: wire 5V to sound chip
Connections:
- wire segments 84 -> 86
Changed lines of the file:
@@
 Text Notes 900  3500 0    118  ~ 0
 7.4 Volts
+Wire Wire Line
+	7400 3400 6800 3400
+Wire Wire Line
+	6800 3400 6800 4350
+Connection ~ 7400 3400
 $EndSCHEMATC

Commit message: switch from WT488D (obsolete) to YX5200
Parts:
- removed A?: WT588D, symbol WT588D
- added A?: YX5200, symbol YX5200
- added R?: 1K, symbol R
Connections:
- wire segments 86 -> 77
Changed lines of the file:
@@
 $EndSheet
-$Comp
-L WT588D A?
-U 1 1 5D7C6302
-P 6200 5050
-F 0 "A?" H 6200 5050 60  0000 C CNN
-F 1 "WT588D" H 6200 4950 60  0000 C TNN
-F 2 "" H 6200 5050 60  0000 C CNN
-F 3 "" H 6200 5050 60  0000 C CNN
-	1    6200 5050
-	1    0    0    -1
-$EndComp
 $Comp
 L Speaker LS?
 U 1 1 5D7C69A9
-P 5300 4550
-F 0 "LS?" H 5350 4775 50  0000 R CNN
-F 1 "Speaker" H 5350 4700 50  0000 R CNN
-F 2 "" H 5300 4350 50  0001 C CNN
-F 3 "" H 5290 4500 50  0001 C CNN
-	1    5300 4550
+P 5400 4500
+F 0 "LS?" H 5450 4725 50  0000 R CNN
+F 1 "Speaker" H 5450 4650 50  0000 R CNN
+F 2 "" H 5400 4300 50  0001 C CNN
+F 3 "" H 5390 4450 50  0001 C CNN
+	1    5400 4500
 	-1   0    0    -1
 $EndComp
@@
 Connection ~ 9850 1850
 Wire Wire Line
-	5500 4550 5600 4550
-Wire Wire Line
-	5500 4650 5600 4650
-Wire Wire Line
-	5600 5050 5600 6400
-Connection ~ 5600 6400
-Wire Wire Line
-	7500 5700 7500 4750
-Wire Wire Line
-	7500 4750 6800 4750
-Wire Wire Line
-	7300 5550 7300 4850
-Wire Wire Line
-	7300 4850 6800 4850
-Wire Wire Line
-	7100 5400 7100 4950
-Wire Wire Line
-	7100 4950 6800 4950
-Wire Wire Line
-	6800 4450 7700 4450
-Wire Wire Line
-	7700 4450 7700 5850
-Wire Wire Line
-	6550 3000 7000 3000
-Wire Wire Line
-	7000 3000 7000 4550
-Wire Wire Line
-	7000 4550 6800 4550
-Wire Wire Line
 	7400 3800 3600 3800
 Connection ~ 3600 3800
@@
 	6550 2000 7400 2000
 Wire Wire Line
-	7400 950  7400 3400
-Wire Wire Line
-	3200 950  7400 950
+	7400 3400 7400 950
+Wire Wire Line
+	7400 950  3200 950
 Connection ~ 7400 2000
 Connection ~ 3800 3800
 Connection ~ 4000 3800
 Wire Wire Line
-	7300 4450 7300 3800
-Connection ~ 7300 3800
-Connection ~ 7300 4450
-Wire Wire Line
-	4950 5400 4950 3100
-Wire Wire Line
-	7100 5400 4950 5400
-Wire Wire Line
-	4950 3100 5350 3100
-Wire Wire Line
-	4850 5550 4850 3000
-Wire Wire Line
-	7300 5550 4850 5550
-Wire Wire Line
-	4850 3000 5350 3000
-Wire Wire Line
-	4750 5700 4750 2900
-Wire Wire Line
-	4750 5700 7500 5700
-Wire Wire Line
-	4750 2900 5350 2900
-Wire Wire Line
-	4650 5850 4650 2800
-Wire Wire Line
 	4650 2800 5350 2800
-Wire Wire Line
-	7700 5850 4650 5850
 Wire Wire Line
 	4200 1100 4200 950
@@
 Text Notes 900  3500 0    118  ~ 0
 7.4 Volts
-Wire Wire Line
-	7400 3400 6800 3400
-Wire Wire Line
-	6800 3400 6800 4350
 Connection ~ 7400 3400
+$Comp
+L YX5200 A?
+U 1 1 5D90CF9F
+P 6400 4600
+F 0 "A?" H 6400 4500 60  0000 C CNN
+F 1 "YX5200" H 6400 4400 60  0000 C TNN
+F 2 "" H 6400 4600 60  0000 C CNN
+F 3 "" H 6400 4600 60  0000 C CNN
+	1    6400 4600
+	1    0    0    -1
+$EndComp
+Wire Wire Line
+	7400 3400 5750 3400
+Wire Wire Line
+	5750 3400 5750 3900
+Wire Wire Line
+	5750 3900 5800 3900
+Wire Wire Line
+	7000 4500 7050 4500
+Wire Wire Line
+	7050 4500 7050 6400
+Connection ~ 7050 6400
+Wire Wire Line
+	4950 4000 5800 4000
+Wire Wire Line
+	4850 4100 5800 4100
+Wire Wire Line
+	5800 4600 5600 4600
+Wire Wire Line
+	5600 4500 5700 4500
+Wire Wire Line
+	5700 4500 5700 4400
+Wire Wire Line
+	5700 4400 5800 4400
+$Comp
+L R R?
+U 1 1 5D915A72
+P 4950 3500
+F 0 "R?" V 5030 3500 50  0000 C CNN
+F 1 "1K" V 4950 3500 50  0000 C CNN
+F 2 "" V 4880 3500 50  0001 C CNN
+F 3 "" H 4950 3500 50  0001 C CNN
+	1    4950 3500
+	1    0    0    -1
+$EndComp
+Wire Wire Line
+	4850 2900 4850 4100
+Wire Wire Line
+	4950 3000 4950 3350
+Wire Wire Line
+	4950 3650 4950 4000
+Wire Wire Line
+	5350 3000 4950 3000
+Wire Wire Line
+	5350 2900 4850 2900
+Wire Wire Line
+	7000 3900 7000 3700
+Wire Wire Line
+	7000 3700 5350 3700
+Wire Wire Line
+	5350 3700 5350 3100
 $EndSCHEMATC

Commit message: update schematic for 'Extra' button
Connections:
- wire segments 77 -> 76
Other:
- note added: "D04 = Trigger"
- note added: "D05 = Yellow"
- note added: "D06 = Green"
- note added: "D07 = Black"
- note added: "D08 = Extra"
Changed lines of the file:
@@
 Sheet 1 2
 Title "Rubber Band Gun"
-Date "2019-09-13"
+Date "2020-01-02"
 Rev "---"
 Comp ""
@@
 Connection ~ 3800 3800
 Connection ~ 4000 3800
-Wire Wire Line
-	4650 2800 5350 2800
 Wire Wire Line
 	4200 1100 4200 950
@@
 Wire Wire Line
 	5350 3700 5350 3100
+Text Notes 2200 2300 0    60   ~ 0
+D04 = Trigger
+Text Notes 2200 2400 0    59   ~ 0
+D05 = Yellow
+Text Notes 2200 2500 0    59   ~ 0
+D06 = Green
+Text Notes 2200 2600 0    59   ~ 0
+D07 = Black
+Text Notes 2200 2700 0    59   ~ 0
+D08 = Extra
 $EndSCHEMATC

Commit message: start work on 3-button version
Parts:
- removed SW? (x2): SW_PUSH, symbol SW_Push
- added SW?: SW_SPST, symbol SW_SPST
- added SW?: SW_PUSH, symbol SW_Push
Other:
- note added: "D09 = Barrel\n grounded = closed"
- note removed: "D08 = Extra"
Changed lines of the file:
@@
-$EndComp
-$Comp
-L SW_Push SW?
-U 1 1 5D7D1785
-P 4200 5050
-F 0 "SW?" H 4350 5160 50  0000 C CNN
-F 1 "SW_PUSH" H 4200 4970 50  0000 C CNN
-F 2 "" H 4200 5050 60  0000 C CNN
-F 3 "" H 4200 5050 60  0000 C CNN
-	1    4200 5050
-	0    -1   -1   0
 $EndComp
 $Comp
@@
 $EndComp
 $Comp
-L SW_Push SW?
-U 1 1 5D7D389D
-P 4400 4300
-F 0 "SW?" H 4550 4410 50  0000 C CNN
-F 1 "SW_PUSH" H 4400 4220 50  0000 C CNN
-F 2 "" H 4400 4300 60  0000 C CNN
-F 3 "" H 4400 4300 60  0000 C CNN
-	1    4400 4300
-	0    -1   -1   0
-$EndComp
-$Comp
 L L L?
 U 1 1 5D7D3BAD
@@
 	5350 2300 3600 2300
 Wire Wire Line
-	3600 1400 3600 4000
+	3600 1400 3600 4100
 Wire Wire Line
 	5350 2400 3800 2400
 Wire Wire Line
-	3800 1400 3800 4700
+	3800 1400 3800 4800
 Wire Wire Line
 	5350 2500 4000 2500
 Wire Wire Line
-	4000 1400 4000 4000
-Wire Wire Line
-	3600 4600 3600 6400
+	4000 1400 4000 4100
+Wire Wire Line
+	3600 4500 3600 6400
 Connection ~ 3600 6400
 Wire Wire Line
-	3800 5300 3800 6400
+	3800 5200 3800 6400
 Connection ~ 3800 6400
 Wire Wire Line
-	4000 4600 4000 6400
+	4000 4500 4000 6400
 Connection ~ 4000 6400
 Wire Wire Line
@@
 Connection ~ 4200 950
 Wire Wire Line
-	4200 1400 4200 4850
-Wire Wire Line
-	4200 5250 4200 6400
-Connection ~ 4200 6400
-Wire Wire Line
 	5350 2600 4200 2600
 Connection ~ 4200 2600
@@
 Connection ~ 4400 950
 Wire Wire Line
-	4400 1400 4400 4100
-Wire Wire Line
-	4400 4500 4400 6400
-Connection ~ 4400 6400
-Wire Wire Line
-	5350 2700 4400 2700
-Connection ~ 4400 2700
+	4400 1400 4400 4500
 Wire Notes Line
 	8350 2550 8350 2850
@@
 Text Notes 2200 2600 0    59   ~ 0
 D07 = Black
-Text Notes 2200 2700 0    59   ~ 0
-D08 = Extra
+Text Notes 2200 2900 0    59   ~ 0
+D09 = Barrel\n    grounded = closed
+Wire Wire Line
+	5350 2800 4400 2800
+Connection ~ 4400 2800
+$Comp
+L SW_SPST SW?
+U 1 1 5E2283C4
+P 4600 4500
+F 0 "SW?" H 4600 4625 50  0000 C CNN
+F 1 "SW_SPST" H 4600 4400 50  0000 C CNN
+F 2 "" H 4600 4500 50  0001 C CNN
+F 3 "" H 4600 4500 50  0001 C CNN
+	1    4600 4500
+	1    0    0    -1
+$EndComp
+Connection ~ 4200 6400
+Wire Wire Line
+	4800 4500 4800 6400
+Connection ~ 4800 6400
+$Comp
+L SW_Push SW?
+U 1 1 5E22B63A
+P 4200 5000
+F 0 "SW?" H 4350 5110 50  0000 C CNN
+F 1 "SW_PUSH" H 4200 4920 50  0000 C CNN
+F 2 "" H 4200 5000 60  0000 C CNN
+F 3 "" H 4200 5000 60  0000 C CNN
+	1    4200 5000
+	0    -1   -1   0
+$EndComp
+Wire Wire Line
+	4200 1400 4200 4800
+Wire Wire Line
+	4200 5200 4200 6400
 $EndSCHEMATC

Commit message: I think it now uses red button OK
Other:
- note added: "D07 = Red"
- note removed: "D07 = Black"
Changed lines of the file:
@@
 Sheet 1 2
 Title "Rubber Band Gun"
-Date "2020-01-02"
+Date "2020-01-18"
 Rev "---"
 Comp ""
@@
 D06 = Green
 Text Notes 2200 2600 0    59   ~ 0
-D07 = Black
+D07 = Red
 Text Notes 2200 2900 0    59   ~ 0
 D09 = Barrel\n    grounded = closed
