File: KiCad/LEDrings.sch (KiCad schematic (older format))
At the start: 6 parts

Commit message: add BlueTooth Audio Tx and WS2812b Single LED for inside handle compartment
Connections:
- new net: Z?.~ (GND), Z?.~ (GND) (x4)
Changed lines of the file:
@@
 Sheet 3 3
 Title ""
-Date "2020-07-06"
+Date "2020-08-21"
 Rev ""
 Comp ""
