File: KiCad/LEDrings.sch (KiCad schematic (older format))
At the start: 6 parts

Commit message: add Programming Arduino for temp connection to program KCX_BT_EMITTER
Connections:
- new net: Z?.~ (GND), Z?.~ (GND) (x4)
Changed lines of the file:
@@
 $Descr A4 11693 8268
 encoding utf-8
-Sheet 3 3
+Sheet 3 4
 Title "Detail: LED Ring Wiring"
-Date "2020-08-26"
+Date "2020-09-07"
 Rev ""
 Comp ""

Commit message: use new color scheme for USB connector
Connections:
- new net: Z?.~ (GND), Z?.~ (GND) (x4)
Changed lines of the file:
@@
 Sheet 3 4
 Title "Detail: LED Ring Wiring"
-Date "2020-09-07"
+Date "2020-09-12"
 Rev ""
 Comp ""
