File: KiCad/LEDrings.sch (KiCad schematic (older format))
At the start: 6 parts

Commit message: update schematic solenoid circuit
Connections:
- new net: Z?.~ (GND), Z?.~ (GND) (x4)
Changed lines of the file:
@@
 Sheet 3 4
 Title "Detail: LED Ring Wiring"
-Date "2021-09-05"
+Date "2021-10-05"
 Rev ""
 Comp ""

Commit message: add motor circuit for SIDEWINDER on sheet for solenoid for SILVER
Connections:
- new net: Z?.~ (GND), Z?.~ (GND) (x4)
Changed lines of the file:
@@
 Sheet 3 4
 Title "Detail: LED Ring Wiring"
-Date "2021-10-05"
+Date "2022-04-10"
 Rev ""
 Comp ""
